Commit message: final updates.

File: slam_project/urdf/udacity_bot.xacro (robot description, xacro)
@@ -146,31 +146,11 @@
     	<child link="camera" />
   	</joint>
- <link name='camera_rgbd_frame'>
-    <visual name='camera_visual'>
-      <origin xyz="0 0 0" rpy=" 0 0 0"/>
-      <geometry>
-        <box size="0.01 0.01 0.01"/>
-      </geometry>
-    </visual>
-    <inertial>
-      <mass value="0.1"/>
-      <origin xyz="0 0 0" rpy=" 0 0 0"/>
-      <inertia
-          ixx="1e-6" ixy="0" ixz="0"
-          iyy="1e-6" iyz="0"
-          izz="1e-6"
-      />
-    </inertial>
-    <collision name='collision'>
-      <origin xyz="0 0 0" rpy=" 0 0 0"/>
-      <geometry>
-        <box size="0.01 0.01 0.01"/>
-      </geometry>
-    </collision>
+ <link name='camera_link_optical'>
   </link>
-  <joint name="camera_joint2" type="fixed">
-    	<origin xyz="0 0 0" rpy="0 0 0" />
+  <joint name="camera_optical_joint" type="fixed">
+    	<!-- <origin xyz="0.3 0 0" rpy="${-pi/2} 0 ${-pi/2}" /> -->
+        <origin xyz="0.3 0 0" rpy="0 0 0" />
     	<parent link="camera"/>
-    	<child link="camera_rgbd_frame" />
+    	<child link="camera_link_optical" />
   	</joint>
   <link name='hokuyo'>

Commit message: final commit.

File: slam_project/urdf/udacity_bot.xacro (robot description, xacro)
@@ -149,6 +149,6 @@
   </link>
   <joint name="camera_optical_joint" type="fixed">
-    	<!-- <origin xyz="0.3 0 0" rpy="${-pi/2} 0 ${-pi/2}" /> -->
-        <origin xyz="0.3 0 0" rpy="0 0 0" />
+    	<origin xyz="0.3 0 0" rpy="${-pi/2} 0 ${-pi/2}" />
+        <!-- <origin xyz="0.3 0 0" rpy="0 0 0" /> -->
     	<parent link="camera"/>
     	<child link="camera_link_optical" />
